Commit message: 1/4

File: ros2_ws/install/my_four_wheel_robot/share/my_four_wheel_robot/urdf/my_robot.urdf.xacro (robot description, xacro)
@@ -1 +1 @@
-/home/bao/ros2_ws/src/my_four_wheel_robot/urdf/my_robot.urdf.xacro
+/home/bao/NCKH-25-26/ros2_ws/src/my_four_wheel_robot/urdf/my_robot.urdf.xacro

File: ros2_ws/src/my_four_wheel_robot/urdf/my_robot.urdf.xacro (robot description, xacro)
@@ -1,15 +1,24 @@
 <?xml version="1.0"?>
 <robot xmlns:xacro="http://ros.org/wiki/xacro" name="my_robot">
-  <!-- ================== THAM SỐ CHUNG - DỄ CHỈNH SỬA Ở ĐÂY ================== -->
-  <xacro:property name="base_length" value="0.5"/>      <!-- dài thân xe (x) -->
-  <xacro:property name="base_width" value="0.4"/>       <!-- rộng thân xe (y) -->
-  <xacro:property name="base_height" value="0.1"/>      <!-- cao thân xe (z) -->
-  <xacro:property name="wheel_radius" value="0.05"/>    <!-- bán kính bánh -->
-  <xacro:property name="wheel_width" value="0.03"/>     <!-- chiều rộng bánh -->
-  <xacro:property name="wheel_mass" value="0.5"/>       <!-- khối lượng mỗi bánh -->
-  <!-- Khoảng cách bánh xe - chỉnh ở đây để thay đổi vị trí bánh -->
-  <xacro:property name="wheel_x_offset" value="0.2"/>      <!-- khoảng cách từ tâm đến trục trước/sau (0.2m) -->
-  <xacro:property name="wheel_separation" value="0.4"/>    <!-- khoảng cách trái-phải giữa hai bánh cùng trục -->
-  <!-- ================== BASE_LINK (thân xe) ================== -->
+  <!-- ========================================================= -->
+  <!-- ARGUMENT NHẬN TỪ FILE LAUNCH                              -->
+  <!-- ========================================================= -->
+  <xacro:arg name="controllers_file" default=""/>
+  <!-- ========================================================= -->
+  <!-- THAM SỐ CHUNG                                             -->
+  <!-- ========================================================= -->
+  <xacro:property name="base_length" value="0.5"/>
+  <xacro:property name="base_width" value="0.4"/>
+  <xacro:property name="base_height" value="0.1"/>
+  <xacro:property name="wheel_radius" value="0.1"/>
+  <xacro:property name="wheel_width" value="0.03"/>
+  <xacro:property name="wheel_mass" value="0.5"/>
+  <xacro:property name="camera_offset_x" value="0.15"/>
+  <xacro:property name="imu_offset_z" value="0.02"/>
+  <xacro:property name="wheel_x_offset" value="0.2"/>
+  <xacro:property name="wheel_separation" value="0.4"/>
+  <!-- ========================================================= -->
+  <!-- BASE                                                      -->
+  <!-- ========================================================= -->
   <link name="base_link">
     <visual>
@@ -17,8 +26,12 @@
         <box size="${base_length} ${base_width} ${base_height}"/>
       </geometry>
-      <material name="blue"><color rgba="0 0 1 1"/></material>
-    </visual>
-    <collision>
-      <geometry><box size="${base_length} ${base_width} ${base_height}"/></geometry>
+      <material name="blue">
+        <color rgba="0 0 1 1"/>
+      </material>
+    </visual>
+    <collision>
+      <geometry>
+        <box size="${base_length} ${base_width} ${base_height}"/>
+      </geometry>
     </collision>
     <inertial>
@@ -27,21 +40,28 @@
     </inertial>
   </link>
-   <link name="base_footprint"/>
-   <joint name="base_joint" type="fixed">
-     <parent link="base_footprint"/>
-     <child link="base_link"/>
+  <link name="base_footprint"/>
+  <joint name="base_joint" type="fixed">
+    <parent link="base_footprint"/>
+    <child link="base_link"/>
     <origin xyz="0 0 0" rpy="0 0 0"/>
   </joint>
-  <!-- ================== 4 BÁNH XE - VIẾT RIÊNG TỪNG CÁI ĐỂ DỄ SỬA ================== -->
-  <!-- BÁNH TRƯỚC TRÁI -->
+  <!-- ========================================================= -->
+  <!-- BÁNH TRƯỚC TRÁI                                           -->
+  <!-- ========================================================= -->
   <link name="left_front_wheel">
     <visual>
       <origin rpy="1.5708 0 0" xyz="0 0 0"/>
-      <geometry><cylinder radius="${wheel_radius}" length="${wheel_width}"/></geometry>
-      <material name="black"><color rgba="0 0 0 1"/></material>
-    </visual>
-    <collision>
-      <origin rpy="1.5708 0 0" xyz="0 0 0"/>
-      <geometry><cylinder radius="${wheel_radius}" length="${wheel_width}"/></geometry>
+      <geometry>
+        <cylinder radius="${wheel_radius}" length="${wheel_width}"/>
+      </geometry>
+      <material name="black">
+        <color rgba="0 0 0 1"/>
+      </material>
+    </visual>
+    <collision>
+      <origin rpy="1.5708 0 0" xyz="0 0 0"/>
+      <geometry>
+        <cylinder radius="${wheel_radius}" length="${wheel_width}"/>
+      </geometry>
     </collision>
     <inertial>
@@ -53,19 +73,25 @@
     <parent link="base_link"/>
     <child link="left_front_wheel"/>
-    <!-- Vị trí bánh trước trái - chỉnh 3 số xyz ở đây -->
-    <origin xyz="${wheel_x_offset} ${wheel_separation/2.0} ${-(base_height/2.0 - wheel_radius)}" rpy="0 0 0"/>
+    <origin xyz="${wheel_x_offset} ${wheel_separation/2.0} ${-(base_height/2.0 + wheel_radius)}" rpy="0 0 0"/>
     <axis xyz="0 1 0"/>
   </joint>
-  <!-- BÁNH TRƯỚC PHẢI -->
+  <!-- ========================================================= -->
+  <!-- BÁNH TRƯỚC PHẢI                                           -->
+  <!-- ========================================================= -->
   <link name="right_front_wheel">
-    <!-- Giống bánh trước trái, chỉ khác tên và vị trí y -->
-    <visual>
-      <origin rpy="1.5708 0 0" xyz="0 0 0"/>
-      <geometry><cylinder radius="${wheel_radius}" length="${wheel_width}"/></geometry>
-      <material name="black"><color rgba="0 0 0 1"/></material>
-    </visual>
-    <collision>
-      <origin rpy="1.5708 0 0" xyz="0 0 0"/>
-      <geometry><cylinder radius="${wheel_radius}" length="${wheel_width}"/></geometry>
+    <visual>
+      <origin rpy="1.5708 0 0" xyz="0 0 0"/>
+      <geometry>
+        <cylinder radius="${wheel_radius}" length="${wheel_width}"/>
+      </geometry>
+      <material name="black">
+        <color rgba="0 0 0 1"/>
+      </material>
+    </visual>
+    <collision>
+      <origin rpy="1.5708 0 0" xyz="0 0 0"/>
+      <geometry>
+        <cylinder radius="${wheel_radius}" length="${wheel_width}"/>
+      </geometry>
     </collision>
     <inertial>
@@ -77,19 +103,25 @@
     <parent link="base_link"/>
     <child link="right_front_wheel"/>
-    <!-- Vị trí bánh trước phải - chỉ thay dấu y -->
-    <origin xyz="${wheel_x_offset} ${-wheel_separation/2.0} ${-(base_height/2.0 - wheel_radius)}" rpy="0 0 0"/>
+    <origin xyz="${wheel_x_offset} ${-wheel_separation/2.0} ${-(base_height/2.0 + wheel_radius)}" rpy="0 0 0"/>
     <axis xyz="0 1 0"/>
   </joint>
-  <!-- BÁNH SAU TRÁI -->
+  <!-- ========================================================= -->
+  <!-- BÁNH SAU TRÁI                                             -->
+  <!-- ========================================================= -->
   <link name="left_rear_wheel">
-    <!-- Giống bánh trước, chỉ khác vị trí x -->
-    <visual>
-      <origin rpy="1.5708 0 0" xyz="0 0 0"/>
-      <geometry><cylinder radius="${wheel_radius}" length="${wheel_width}"/></geometry>
-      <material name="black"><color rgba="0 0 0 1"/></material>
-    </visual>
-    <collision>
-      <origin rpy="1.5708 0 0" xyz="0 0 0"/>
-      <geometry><cylinder radius="${wheel_radius}" length="${wheel_width}"/></geometry>
+    <visual>
+      <origin rpy="1.5708 0 0" xyz="0 0 0"/>
+      <geometry>
+        <cylinder radius="${wheel_radius}" length="${wheel_width}"/>
+      </geometry>
+      <material name="black">
+        <color rgba="0 0 0 1"/>
+      </material>
+    </visual>
+    <collision>
+      <origin rpy="1.5708 0 0" xyz="0 0 0"/>
+      <geometry>
+        <cylinder radius="${wheel_radius}" length="${wheel_width}"/>
+      </geometry>
     </collision>
     <inertial>
@@ -101,18 +133,25 @@
     <parent link="base_link"/>
     <child link="left_rear_wheel"/>
-    <!-- Vị trí bánh sau trái - x âm -->
-    <origin xyz="${-wheel_x_offset} ${wheel_separation/2.0} ${-(base_height/2.0 - wheel_radius)}" rpy="0 0 0"/>
+    <origin xyz="${-wheel_x_offset} ${wheel_separation/2.0} ${-(base_height/2.0 + wheel_radius)}" rpy="0 0 0"/>
     <axis xyz="0 1 0"/>
   </joint>
-  <!-- BÁNH SAU PHẢI -->
+  <!-- ========================================================= -->
+  <!-- BÁNH SAU PHẢI                                             -->
+  <!-- ========================================================= -->
   <link name="right_rear_wheel">
     <visual>
       <origin rpy="1.5708 0 0" xyz="0 0 0"/>
-      <geometry><cylinder radius="${wheel_radius}" length="${wheel_width}"/></geometry>
-      <material name="black"><color rgba="0 0 0 1"/></material>
-    </visual>
-    <collision>
-      <origin rpy="1.5708 0 0" xyz="0 0 0"/>
-      <geometry><cylinder radius="${wheel_radius}" length="${wheel_width}"/></geometry>
+      <geometry>
+        <cylinder radius="${wheel_radius}" length="${wheel_width}"/>
+      </geometry>
+      <material name="black">
+        <color rgba="0 0 0 1"/>
+      </material>
+    </visual>
+    <collision>
+      <origin rpy="1.5708 0 0" xyz="0 0 0"/>
+      <geometry>
+        <cylinder radius="${wheel_radius}" length="${wheel_width}"/>
+      </geometry>
     </collision>
     <inertial>
@@ -124,26 +163,156 @@
     <parent link="base_link"/>
     <child link="right_rear_wheel"/>
-    <!-- Vị trí bánh sau phải - x âm, y âm -->
-    <origin xyz="${-wheel_x_offset} ${-wheel_separation/2.0} ${-(base_height/2.0 - wheel_radius)}" rpy="0 0 0"/>
+    <origin xyz="${-wheel_x_offset} ${-wheel_separation/2.0} ${-(base_height/2.0 + wheel_radius)}" rpy="0 0 0"/>
     <axis xyz="0 1 0"/>
   </joint>
-  <!-- ================== ros2_control (giữ nguyên nhưng dùng tên mới cho Jazzy) ================== -->
+  <!-- ========================================================= -->
+  <!-- GAZEBO CONTACT / FRICTION                                 -->
+  <!-- ========================================================= -->
+  <gazebo reference="left_front_wheel">
+    <mu1>1.0</mu1>
+    <mu2>0.8</mu2>
+    <kp>1e8</kp>
+    <kd>1</kd>
+    <min_depth>0.001</min_depth>
+  </gazebo>
+  <gazebo reference="right_front_wheel">
+    <mu1>1.0</mu1>
+    <mu2>0.8</mu2>
+    <kp>1e8</kp>
+    <kd>1</kd>
+    <min_depth>0.001</min_depth>
+  </gazebo>
+  <gazebo reference="left_rear_wheel">
+    <mu1>1.0</mu1>
+    <mu2>0.8</mu2>
+    <kp>1e8</kp>
+    <kd>1</kd>
+    <min_depth>0.001</min_depth>
+  </gazebo>
+  <gazebo reference="right_rear_wheel">
+    <mu1>1.0</mu1>
+    <mu2>0.8</mu2>
+    <kp>1e8</kp>
+    <kd>1</kd>
+    <min_depth>0.001</min_depth>
+  </gazebo>
+  <!-- ========================================================= -->
+  <!-- ROS2_CONTROL                                              -->
+  <!-- ========================================================= -->
   <ros2_control name="GazeboSimSystem" type="system">
     <hardware>
-      <plugin>gz_ros2_control/GazeboSimSystem</plugin>  <!-- sửa cho Harmonic -->
+      <plugin>gz_ros2_control/GazeboSimSystem</plugin>
     </hardware>
-    <joint name="left_front_wheel_joint"><command_interface name="velocity"/><state_interface name="position"/><state_interface name="velocity"/></joint>
-    <joint name="left_rear_wheel_joint"><command_interface name="velocity"/><state_interface name="position"/><state_interface name="velocity"/></joint>
-    <joint name="right_front_wheel_joint"><command_interface name="velocity"/><state_interface name="position"/><state_interface name="velocity"/></joint>
-    <joint name="right_rear_wheel_joint"><command_interface name="velocity"/><state_interface name="position"/><state_interface name="velocity"/></joint>
+    <joint name="left_front_wheel_joint">
+      <command_interface name="velocity"/>
+      <state_interface name="position"/>
+      <state_interface name="velocity"/>
+    </joint>
+    <joint name="left_rear_wheel_joint">
+      <command_interface name="velocity"/>
+      <state_interface name="position"/>
+      <state_interface name="velocity"/>
+    </joint>
+    <joint name="right_front_wheel_joint">
+      <command_interface name="velocity"/>
+      <state_interface name="position"/>
+      <state_interface name="velocity"/>
+    </joint>
+    <joint name="right_rear_wheel_joint">
+      <command_interface name="velocity"/>
+      <state_interface name="position"/>
+      <state_interface name="velocity"/>
+    </joint>
   </ros2_control>
-  <!-- Plugin cho Gazebo Harmonic (sửa tên file .so) -->
+  <!-- ========================================================= -->
+  <!-- PLUGIN GZ_ROS2_CONTROL                                    -->
+  <!-- QUAN TRỌNG: dùng ${controllers_file}                      -->
+  <!-- ========================================================= -->
   <gazebo>
     <plugin filename="libgz_ros2_control-system.so" name="gz_ros2_control::GazeboSimROS2ControlPlugin">
-      <parameters>$(find my_four_wheel_robot)/config/my_controller.yaml</parameters>
+      <parameters>$(arg controllers_file)</parameters>
     </plugin>
   </gazebo>
-   <gazebo reference="base_link">
-    <material>Gazebo/Blue</material>
-   </gazebo>
+  <!-- ========================================================= -->
+  <!-- CAMERA                                                    -->
+  <!-- ========================================================= -->
+  <link name="camera_link">
+    <visual>
+      <geometry>
+        <box size="0.06 0.03 0.03"/>
+      </geometry>
+      <material name="black"/>
+    </visual>
+    <collision>
+      <geometry>
+        <box size="0.06 0.03 0.03"/>
+      </geometry>
+    </collision>
+    <inertial>
+      <mass value="0.1"/>
+      <inertia ixx="0.001" ixy="0.0" ixz="0.0" iyy="0.001" iyz="0.0" izz="0.001"/>
+    </inertial>
+  </link>
+  <joint name="camera_joint" type="fixed">
+    <parent link="base_link"/>
+    <child link="camera_link"/>
+    <origin xyz="${camera_offset_x} 0 ${base_height/2}" rpy="0 0 0"/>
+  </joint>
+  <gazebo reference="camera_link">
+    <sensor name="rgb_camera" type="camera">
+      <always_on>true</always_on>
+      <update_rate>30</update_rate>
+      <topic>camera/rgb/image_raw</topic>
+      <camera name="rgb">
+        <horizontal_fov>1.047</horizontal_fov>
+        <image>
+          <width>640</width>
+          <height>480</height>
+          <format>R8G8B8</format>
+        </image>
+        <clip>
+          <near>0.03</near>
+          <far>100</far>
+        </clip>
+      </camera>
+    </sensor>
+    <sensor name="depth_camera" type="depth_camera">
+      <always_on>true</always_on>
+      <update_rate>30</update_rate>
+      <topic>camera/depth/image_raw</topic>
+      <camera name="depth">
+        <horizontal_fov>1.047</horizontal_fov>
+        <image>
+          <width>640</width>
+          <height>480</height>
+        </image>
+        <clip>
+          <near>0.03</near>
+          <far>10.0</far>
+        </clip>
+      </camera>
+    </sensor>
+  </gazebo>
+  <!-- ========================================================= -->
+  <!-- IMU                                                       -->
+  <!-- ========================================================= -->
+  <link name="imu_link">
+    <inertial>
+      <mass value="0.01"/>
+      <inertia ixx="0.0001" ixy="0.0" ixz="0.0" iyy="0.0001" iyz="0.0" izz="0.0001"/>
+    </inertial>
+  </link>
+  <joint name="imu_joint" type="fixed">
+    <parent link="base_link"/>
+    <child link="imu_link"/>
+    <origin xyz="0 0 ${base_height + imu_offset_z}" rpy="0 0 0"/>
+  </joint>
+  <gazebo reference="imu_link">
+    <sensor name="imu_sensor" type="imu">
+      <always_on>true</always_on>
+      <update_rate>100</update_rate>
+      <topic>imu</topic>
+      <imu/>
+    </sensor>
+  </gazebo>
 </robot>
