Commit message: 16/5

File: Rocker-Bogie/install/six_ws_robot/share/six_ws_robot/urdf/six_ws_robot.xacro (robot description, xacro)
@@ -111,8 +111,15 @@
     <origin xyz="${camera_offset_x} 0 ${camera_offset_z}" rpy="0 0 0"/>
   </joint>
+  <!-- Optical frame: Z forward, X right, Y down (camera convention) -->
+  <link name="camera_optical_link"/>
+  <joint name="camera_optical_joint" type="fixed">
+    <parent link="camera_link"/>
+    <child link="camera_optical_link"/>
+    <origin xyz="0 0 0" rpy="${-pi/2} 0 ${-pi/2}"/>
+  </joint>
   <gazebo reference="camera_link">
     <sensor name="rgb_camera" type="camera">
       <always_on>true</always_on>
-      <update_rate>30</update_rate>
+      <update_rate>15</update_rate>
       <visualize>true</visualize>
       <topic>camera/rgb/image_raw</topic>
@@ -128,4 +135,5 @@
           <far>50.0</far>
         </clip>
+        <optical_frame_id>camera_optical_link</optical_frame_id>
       </camera>
     </sensor>
@@ -145,7 +153,9 @@
           <far>20.0</far>
         </clip>
+        <optical_frame_id>camera_optical_link</optical_frame_id>
       </camera>
     </sensor>
   </gazebo>
+  <!-- IMU Link
   <link name="imu_link">
     <visual>
@@ -176,5 +186,5 @@
       <imu/>
     </sensor>
-  </gazebo>
+  </gazebo> -->
   <ros2_control name="GazeboSimSystem" type="system">
     <hardware>

Commit message: xe chay dc tui

File: Rocker-Bogie/install/six_ws_robot/share/six_ws_robot/urdf/six_ws_robot.xacro (robot description, xacro)
@@ -1,235 +1 @@
-<?xml version="1.0"?>
-<robot xmlns:xacro="http://www.ros.org/wiki/xacro" name="six_ws_robot">
-  <xacro:arg name="controllers_file" default=""/>
-  <xacro:property name="base_length" value="1.00"/>
-  <xacro:property name="base_width" value="0.60"/>
-  <xacro:property name="base_height" value="0.20"/>
-  <xacro:property name="base_mass" value="25.0"/>
-  <xacro:property name="wheel_radius" value="0.15"/>
-  <xacro:property name="wheel_width" value="0.06"/>
-  <xacro:property name="wheel_mass" value="1.0"/>
-  <!-- Drop axle below body so wheels are clearly outside the chassis in RViz/Gazebo -->
-  <xacro:property name="wheel_axle_drop" value="0.06"/>
-  <xacro:property name="wheel_z_offset" value="${-(base_height * 0.5 + wheel_axle_drop)}"/>
-  <xacro:property name="camera_offset_x" value="0.32"/>
-  <xacro:property name="camera_offset_z" value="0.18"/>
-  <xacro:property name="imu_offset_z" value="0.14"/>
-  <link name="base_footprint"/>
-  <joint name="base_footprint_joint" type="fixed">
-    <parent link="base_footprint"/>
-    <child link="base_link"/>
-    <origin xyz="0 0 ${wheel_radius + base_height * 0.5 + wheel_axle_drop}" rpy="0 0 0"/>
-  </joint>
-  <link name="base_link">
-    <visual>
-      <geometry>
-        <box size="${base_length} ${base_width} ${base_height}"/>
-      </geometry>
-      <material name="body_gray">
-        <color rgba="0.35 0.35 0.38 1.0"/>
-      </material>
-    </visual>
-    <collision>
-      <geometry>
-        <box size="${base_length} ${base_width} ${base_height}"/>
-      </geometry>
-    </collision>
-    <inertial>
-      <origin xyz="0 0 0" rpy="0 0 0"/>
-      <mass value="${base_mass}"/>
-      <inertia ixx="1.0" ixy="0.0" ixz="0.0" iyy="1.8" iyz="0.0" izz="2.0"/>
-    </inertial>
-  </link>
-  <xacro:macro name="wheel_module" params="name x y">
-    <link name="${name}_wheel_link">
-      <visual>
-        <origin xyz="0 0 0" rpy="1.5708 0 0"/>
-        <geometry>
-          <cylinder radius="${wheel_radius}" length="${wheel_width}"/>
-        </geometry>
-        <material name="wheel_black">
-          <color rgba="0.08 0.08 0.08 1.0"/>
-        </material>
-      </visual>
-      <collision>
-        <origin xyz="0 0 0" rpy="1.5708 0 0"/>
-        <geometry>
-          <cylinder radius="${wheel_radius}" length="${wheel_width}"/>
-        </geometry>
-      </collision>
-      <inertial>
-        <origin xyz="0 0 0" rpy="0 0 0"/>
-        <mass value="${wheel_mass}"/>
-        <inertia ixx="0.01" ixy="0.0" ixz="0.0" iyy="0.01" iyz="0.0" izz="0.01"/>
-      </inertial>
-    </link>
-    <joint name="${name}_wheel_joint" type="continuous">
-      <parent link="base_link"/>
-      <child link="${name}_wheel_link"/>
-      <origin xyz="${x} ${y} ${wheel_z_offset}" rpy="0 0 0"/>
-      <axis xyz="0 1 0"/>
-      <limit effort="60" velocity="35"/>
-      <dynamics damping="0.2" friction="0.1"/>
-    </joint>
-    <gazebo reference="${name}_wheel_link">
-      <mu1>1.4</mu1>
-      <mu2>1.2</mu2>
-      <kp>1000000.0</kp>
-      <kd>10.0</kd>
-      <min_depth>0.001</min_depth>
-    </gazebo>
-  </xacro:macro>
-  <xacro:wheel_module name="lf" x="0.40" y="0.30"/>
-  <xacro:wheel_module name="lm" x="0.00" y="0.30"/>
-  <xacro:wheel_module name="lr" x="-0.40" y="0.30"/>
-  <xacro:wheel_module name="rf" x="0.40" y="-0.30"/>
-  <xacro:wheel_module name="rm" x="0.00" y="-0.30"/>
-  <xacro:wheel_module name="rr" x="-0.40" y="-0.30"/>
-  <link name="camera_link">
-    <visual>
-      <geometry>
-        <box size="0.08 0.04 0.04"/>
-      </geometry>
-      <material name="sensor_dark">
-        <color rgba="0.12 0.12 0.14 1.0"/>
-      </material>
-    </visual>
-    <collision>
-      <geometry>
-        <box size="0.08 0.04 0.04"/>
-      </geometry>
-    </collision>
-    <inertial>
-      <origin xyz="0 0 0" rpy="0 0 0"/>
-      <mass value="0.15"/>
-      <inertia ixx="0.001" ixy="0.0" ixz="0.0" iyy="0.001" iyz="0.0" izz="0.001"/>
-    </inertial>
-  </link>
-  <joint name="camera_joint" type="fixed">
-    <parent link="base_link"/>
-    <child link="camera_link"/>
-    <origin xyz="${camera_offset_x} 0 ${camera_offset_z}" rpy="0 0 0"/>
-  </joint>
-  <!-- Optical frame: Z forward, X right, Y down (camera convention) -->
-  <link name="camera_optical_link"/>
-  <joint name="camera_optical_joint" type="fixed">
-    <parent link="camera_link"/>
-    <child link="camera_optical_link"/>
-    <origin xyz="0 0 0" rpy="${-pi/2} 0 ${-pi/2}"/>
-  </joint>
-  <gazebo reference="camera_link">
-    <sensor name="rgb_camera" type="camera">
-      <always_on>true</always_on>
-      <update_rate>15</update_rate>
-      <visualize>true</visualize>
-      <topic>camera/rgb/image_raw</topic>
-      <camera name="rgb">
-        <horizontal_fov>1.047</horizontal_fov>
-        <image>
-          <width>640</width>
-          <height>480</height>
-          <format>R8G8B8</format>
-        </image>
-        <clip>
-          <near>0.05</near>
-          <far>50.0</far>
-        </clip>
-        <optical_frame_id>camera_optical_link</optical_frame_id>
-      </camera>
-    </sensor>
-    <sensor name="depth_camera" type="depth_camera">
-      <always_on>true</always_on>
-      <update_rate>15</update_rate>
-      <visualize>true</visualize>
-      <topic>camera/depth/image_raw</topic>
-      <camera name="depth">
-        <horizontal_fov>1.047</horizontal_fov>
-        <image>
-          <width>640</width>
-          <height>480</height>
-        </image>
-        <clip>
-          <near>0.05</near>
-          <far>20.0</far>
-        </clip>
-        <optical_frame_id>camera_optical_link</optical_frame_id>
-      </camera>
-    </sensor>
-  </gazebo>
-  <!-- IMU Link
-  <link name="imu_link">
-    <visual>
-      <geometry>
-        <sphere radius="0.02"/>
-      </geometry>
-      <material name="imu_red">
-        <color rgba="0.8 0.2 0.2 1.0"/>
-      </material>
-    </visual>
-    <inertial>
-      <origin xyz="0 0 0" rpy="0 0 0"/>
-      <mass value="0.02"/>
-      <inertia ixx="0.0001" ixy="0.0" ixz="0.0" iyy="0.0001" iyz="0.0" izz="0.0001"/>
-    </inertial>
-  </link>
-  <joint name="imu_joint" type="fixed">
-    <parent link="base_link"/>
-    <child link="imu_link"/>
-    <origin xyz="0 0 ${imu_offset_z}" rpy="0 0 0"/>
-  </joint>
-  <gazebo reference="imu_link">
-    <sensor name="body_imu" type="imu">
-      <always_on>true</always_on>
-      <update_rate>100</update_rate>
-      <visualize>false</visualize>
-      <topic>imu</topic>
-      <imu/>
-    </sensor>
-  </gazebo> -->
-  <ros2_control name="GazeboSimSystem" type="system">
-    <hardware>
-      <plugin>gz_ros2_control/GazeboSimSystem</plugin>
-    </hardware>
-    <joint name="lf_wheel_joint">
-      <command_interface name="velocity"/>
-      <state_interface name="position"/>
-      <state_interface name="velocity"/>
-      <state_interface name="effort"/>
-    </joint>
-    <joint name="lm_wheel_joint">
-      <command_interface name="velocity"/>
-      <state_interface name="position"/>
-      <state_interface name="velocity"/>
-      <state_interface name="effort"/>
-    </joint>
-    <joint name="lr_wheel_joint">
-      <command_interface name="velocity"/>
-      <state_interface name="position"/>
-      <state_interface name="velocity"/>
-      <state_interface name="effort"/>
-    </joint>
-    <joint name="rf_wheel_joint">
-      <command_interface name="velocity"/>
-      <state_interface name="position"/>
-      <state_interface name="velocity"/>
-      <state_interface name="effort"/>
-    </joint>
-    <joint name="rm_wheel_joint">
-      <command_interface name="velocity"/>
-      <state_interface name="position"/>
-      <state_interface name="velocity"/>
-      <state_interface name="effort"/>
-    </joint>
-    <joint name="rr_wheel_joint">
-      <command_interface name="velocity"/>
-      <state_interface name="position"/>
-      <state_interface name="velocity"/>
-      <state_interface name="effort"/>
-    </joint>
-  </ros2_control>
-  <gazebo>
-    <plugin filename="gz_ros2_control-system" name="gz_ros2_control::GazeboSimROS2ControlPlugin">
-      <parameters>$(arg controllers_file)</parameters>
-    </plugin>
-  </gazebo>
-</robot>
+/home/bao/NCKH-25-26/Rocker-Bogie/src/urdf/six_ws_robot.xacro
